File: pcb/Telemetrie v2.kicad_sch (KiCad schematic)
At the start: 68 parts, among them J1 Conn_02x03_Odd_Even, J2 Conn_01x02_Pin, J3 CONSMA001-SMD-G-T, J4 Conn_01x04_Pin, J5 Conn_01x02_Pin, M1 Conn_01x01_Pin, M2 Conn_01x01_Pin, M3 Conn_01x01_Pin, M4 Conn_01x01_Pin, U1 AVR128DB64x-xPT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

Commit message: update pcb
Parts:
- added D13, D14, D15, D16: LED, LED_SMD:LED_0805_2012Metric_Pad1.15x1.40mm_HandSolder, symbol Device:LED
- added R13, R14, R15, R16: 100R, Resistor_SMD:R_0805_2012Metric_Pad1.20x1.40mm_HandSolder, symbol Device:R
- renumbered R15 to R17, R16 to R18, R13 to R19, R14 to R20
Connections:
- net +3V3: now also D13.2 (A), D14.2 (A), D15.2 (A), D16.2 (A)
- net RX4: now also R16.1
- net RXD: now also R13.2
- net TX4: now also R15.2
- net TXD: now also R14.1
- new net: D16.1 (K), R16.2
- new net: D14.1 (K), R14.2
- new net: D13.1 (K), R13.1
- new net: D15.1 (K), R15.1

Commit message: silkscreen and schematic update
Parts:
- removed D13, D14: LED, LED_SMD:LED_0805_2012Metric_Pad1.15x1.40mm_HandSolder, symbol Device:LED
- added D3, D4: LED, LED_SMD:LED_0805_2012Metric_Pad1.15x1.40mm_HandSolder, symbol Device:LED
- J3: value CONSMA001-SMD-G-T -> SMA SMD
Connections:
- net +3V3: now also D3.2 (A), D4.2 (A)
- net at R14.2: now also D4.1 (K)
- net at R13.1: now also D3.1 (K)
Other:
- moved on the sheet: C1, C2, C3, C4, C5, D10, D15, D16, D5, D6, D7, D8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

Commit message: update schematic and silkscreen
Parts:
- added TP16, TP17: ~, Footprints:TestPoint, symbol Connector:TestPoint
- renumbered D3 to D13, D4 to D14
Connections:
- net D3: now also TP17.1
- net at C5.1, R17.1, U2.12 (RESET): now also TP16.1
- net RXD renamed TX0
- net TXD renamed RX0
Other:
- moved on the sheet: C1, C2, C3, C4, C5, D10, D13, D14, D15, D16, D5, D6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
