File: groundstation/pcb/Motherboard/TelemetryGroundstationMB.kicad_pcb (KiCad board)
At the start: 2 copper layers, 133 x 79.8 mm, 129 parts, among them J1 USB-C, J10 Conn_01x01, J11 Conn_01x01, J12 USB-C, J2 USB-C, J3 ICD15S13E4GV00LF, J4 USB-C, J5 ICD15S13E4GV00LF, J6 ICD15S13E4GV00LF, J7 ICD15S13E4GV00LF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

Commit message: finishing touches to motherboard
Parts:
- moved D27 2.00 mm to (163.5, 137.4)
- moved D28 2.00 mm to (161.0, 137.4)
- moved D29 2.00 mm to (158.5, 137.4)
- moved D30 2.00 mm to (156.0, 137.4)
- moved D31 2.00 mm to (153.5, 137.4)
- moved D32 2.00 mm to (151.0, 137.4)
- moved D33 2.00 mm to (148.5, 137.4)
- moved D34 2.00 mm to (146.0, 137.4)
- moved R47 2.00 mm to (163.5, 132.4)
- moved R48 2.00 mm to (161.0, 132.4)
- moved R51 2.00 mm to (158.5, 132.4)
- moved R52 2.00 mm to (156.0, 132.4)
- moved R53 2.00 mm to (153.5, 132.4)
- moved R54 2.00 mm to (151.0, 132.4)
- moved R55 2.00 mm to (148.5, 132.4)
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Routing:
- net +5V: track 359.3 -> 362.9 mm

Commit message: improve component 3d models
also update pcb 3d models and renderings. fixes #35
Parts:
- J11: footprint Footprints:Banana_CT3151-0 -> Footprints:Banana_CT3151-2
Changed lines of the file:
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@@
 		(embedded_fonts no)
 	)
-	(footprint "Footprints:Banana_CT3151-0"
+	(footprint "Footprints:Banana_CT3151-2"
 		(layer "F.Cu")
 		(at 104.75 115.75 -90)
@@
 			)
 		)
-		(property "Description" "Generic connector, single row, 01x01, script generated (kicad-library-utils/schlib/autogen/connector/)"
+		(property "Description" ""
 			(at 0 0 270)
 			(unlocked yes)
@@
 		(sheetname "/")
 		(sheetfile "TelemetryGroundstationMB.kicad_sch")
-		(attr smd)
+		(attr through_hole)
 		(fp_rect
 			(start -4 -6.5)
@@
 		)
 		(embedded_fonts no)
-		(model "${KIPRJMOD}/3D Models/CT3151-0.STEP"
+		(model "${KIPRJMOD}/3D Models/CT3151-2.STEP"
 			(offset
 				(xyz 10.5 0 13)

Commit message: fix 3D Models and rearrange wires. Fixes #46
Parts:
- C1, C3, C6: value 4.7 uF -> 4.7u
- C10, C11, C12, C9: value 1 uF -> 1u
- C13: value 100uF Elko -> 100u Elko
- C2, C4, C5: value 0.1 uF -> 0.1u
- C7: value 10uF Tantal -> 10u Tantal
- R1, R11, R12, R17, R2, R20, R21, R25, R26, R3, R37, R4, R47, R48, R5, R51, R52, R53, R54, R55, R56, R6: value 560 Ohm -> 560R
- R18, R19: value 470 Ohm -> 470R
Connections:
- U6 pad 1: GND -> +5V
- U6 pad 2: +5V -> GND
Routing:
- net +5V: track 362.9 -> 360.5 mm
